File: Nikon-GPS.kicad_pcb (KiCad board)
At the start: 4 copper layers, 30 x 30 mm, 79 parts, among them J1 Conn_01x09, J2 USB_C_Receptacle_USB2.0_16P, J3 Conn_Coaxial, J4 Hot-Shoe, J6 DEBUG, Q1 BSS138DW, Q2 BSS138DW, Q3 Si1016X, Q5 BSS138DW, SW1 PWR, SW2 El Button, U1 MAX-M10S, U2 TXU0101, U3 GW J9LHS2.4M-C0C7-2+35+13+40A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, U4 BMD-340, U5 XT25F128F, U6 TPS70933DBV, U7 LSM303AGR, U8 BMP581, U9 USBLC6-2SC6

Commit message: idk
Connections:
- U4 pad 19: unconnected-(U4-P0.03-Pad19) -> /MCU/El_Button
Routing:
- net /MCU/El_Button: track 5.51 -> 32.5 mm, vias 1 -> 2
- net unconnected-(U4-P0.03-Pad19): track 5.08 -> 0.00 mm, vias 1 -> 0
- net GND: track 11.5 -> 14.6 mm, vias 77 -> 76
- net /MCU/Accel_INT: track 24.6 -> 25.6 mm
