File: power.kicad_sch (KiCad schematic)
At the start: 9 parts, among them SW1 PWR, U6 TPS70933DBV

Commit message: idk
Parts:
- C1: LCSC C28323 -> C344178
Changed lines of the file:
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@@
 			)
 		)
-		(property "LCSC" "C28323"
+		(property "LCSC" "C344178"
 			(at 110.49 105.41 0)
 			(hide yes)
