File: sensors.kicad_sch (KiCad schematic)
At the start: 16 parts, among them J3 Conn_Coaxial, Q3 Si1016X, U1 MAX-M10S, U7 LSM303AGR, U8 BMP581

Commit message: idk
Parts:
- U8: value BMP581 -> BMP384; LCSC C5362283 -> C5577555
Changed lines of the file:
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@@
 			)
 		)
-		(property "Value" "BMP581"
+		(property "Value" "BMP384"
 			(at 247.65 109.1498 0)
 			(show_name no)
@@
 			)
 		)
-		(property "LCSC" "C5362283"
+		(property "LCSC" "C5577555"
 			(at 234.95 113.03 0)
 			(hide yes)
